File: HW/NoiStop/NoiStop.kicad_pcb (KiCad board)
At the start: 2 copper layers, 48 x 29 mm, 13 parts, among them J3 RX, J4 TX, J5 GND, U1 ESP32-WROOM-32

Commit message: modificata cartella HW
Parts:
- added J6: VDD, MyPads:CIRC_PAD_0.7x0.3, F.Cu at (153.6, 68.1)
- C3: value 100n -> 1u
Connections:
- net Net-(PS1-AC1) renamed /230V AC
Other:
- board text added: "230V AC+"
- board text added: "230V AC-"
- board text added: "GND"
- board text added: "RX"
- board text added: "TX"
- board text added: "VDD"
