File: HW/NoiStop/NoiStop.kicad_sch (KiCad schematic)
At the start: 13 parts, among them J3 RX, J4 TX, J5 GND, U1 ESP32-WROOM-32

Commit message: modificata cartella HW
Parts:
- added J6: VDD, MyPads:CIRC_PAD_0.7x0.3, symbol MyPads:CIRC_PAD_0.7X0.3
Connections:
- net VDD: now also J6.1
- net 230V AC: now reaches J1.1, PS1.1 (AC1)
Other:
- moved on the sheet: J1
